Commit message: fix some xiaoqiang udrf model buggers

File: cartographer_ros/urdf/rplidar_2d.urdf (robot description, URDF)
Before this commit: robot xiaoqiang_udrf, 6 links, 5 joints
Joints:
- joint rot1: type continuous -> fixed
- joint rot2: type continuous -> fixed
- joint rot3: type continuous -> fixed

Commit message: fix lungu rplidar udrf

File: cartographer_ros/urdf/rplidar_2d.urdf (robot description, URDF)
Before this commit: robot xiaoqiang_udrf, 6 links, 5 joints
Links:
- removed link back_wheel
- removed link laserbase_footprint
- added link base_footprint
- added link front1_wheel, mass 0.126682636045453; collision mesh filename=package://xiaoqiang_udrf/meshes/front1_wheel.STL; visual mesh filename=package://xiaoqiang_udrf/meshes/front1_wheel.STL
- added link front2_wheel, mass 0.126682635871512; collision mesh filename=package://xiaoqiang_udrf/meshes/front2_wheel.STL; visual mesh filename=package://xiaoqiang_udrf/meshes/front2_wheel.STL
- added link imu; visual cylinder length=0.01 radius=0.01
- added link kinect_link, mass 0.588695418123486; collision mesh filename=package://xiaoqiang_udrf/meshes/kinect_link.STL; visual mesh filename=package://xiaoqiang_udrf/meshes/kinect_link.STL
- link laserbase_link: mass 4.3093 -> 8.36303567682231
- link left_wheel: mass 0.4651 -> 0.834069618273221
- link right_wheel: mass 0.4651 -> 0.834069618273221
Joints:
- removed joint laserbase_link_joint
- removed joint rot1
- removed joint rot2
- removed joint rot3
- added joint base_link_joint: type fixed, parent base_footprint, child laserbase_link, origin xyz=0 0 0.15
- added joint imu_link_joint: type fixed, parent laserbase_link, child imu, origin xyz=0 0 0 rpy=0 0 0
- added joint kinect: type fixed, parent laserbase_link, child kinect_link, origin xyz=0.13823 0 0.255 rpy=-1.4803 0 -1.5708
- added joint left_rot: type fixed, parent laserbase_link, child front1_wheel, origin xyz=0.26879 0.0795 -0.02225 rpy=1.5708 0 -2.0971
- added joint left_whell: type fixed, parent laserbase_link, child left_wheel, origin xyz=0 0.137 -0.035 rpy=-1.5708 0.68527 -3.1416
- added joint right_rot: type fixed, parent laserbase_link, child front2_wheel, origin xyz=0.26879 -0.0805 -0.02225 rpy=1.5708 0 -0.38246
- added joint right_wheel: type fixed, parent laserbase_link, child right_wheel, origin xyz=0 -0.137 -0.035 rpy=-1.5708 0.82165 5.3376E-17
