Commit message: fix rslidar params

File: cartographer_ros/urdf/rslidar_2d.urdf (robot description, URDF)
Before this commit: robot xiaoqiang_udrf, 9 links, 8 joints
Links:
- removed link front1_wheel
- removed link front2_wheel
- removed link kinect_link
- added link back_wheel, mass 0.070437; collision mesh filename=package://xiaoqiang_udrf/meshes/back_wheel.STL; visual mesh filename=package://xiaoqiang_udrf/meshes/back_wheel.STL
- link laserbase_link: mass 8.36303567682231 -> 4.3093
- link left_wheel: mass 0.834069618273221 -> 0.4651
- link right_wheel: mass 0.834069618273221 -> 0.4651
Joints:
- removed joint kinect
- removed joint left_rot
- removed joint left_whell
- removed joint right_rot
- removed joint right_wheel
- added joint rot1: type fixed, parent laserbase_link, child right_wheel, origin xyz=0 -0.176 -0.05489 rpy=1.5708 0 0, axis 0 0 -1
- added joint rot2: type fixed, parent laserbase_link, child left_wheel, origin xyz=0 0.176 -0.05489 rpy=-1.5708 0 3.1416, axis 0 0 -1
- added joint rot3: type fixed, parent laserbase_link, child back_wheel, origin xyz=-0.25204 -0.00060998 -0.037 rpy=1.5708 0 -5.9631E-17, axis 0 -1 0
- joint horizontal_laser_link_joint: origin xyz=0 0 0.4 rpy=0 0 0 -> xyz=-0.25 0 0.4 rpy=0 0 0
